File: TRL_fixture_JLC04161H-7628.kicad_pcb (KiCad board)
At the start: 4 copper layers, 100 x 56 mm, 11 parts, among them J1 142-0761-861, J2 142-0761-861, J3 142-0761-861, J4 142-0761-861, J5 142-0761-861, J6 142-0761-861, J7 e, J8 142-0761-861, J9 142-0761-861

Commit message: TRL fixture DRC clean
Parts:
- J7: value e -> 142-0761-861
- moved NT1 0.75 mm to (108.9, 100.8)
- moved J1 0.42 mm to (92.0, 105.2)
- moved J2 0.42 mm to (92.0, 96.8)
- moved J3 0.42 mm to (109.0, 105.2)
- moved J4 0.42 mm to (126.0, 105.2)
- moved J5 0.42 mm to (143.0, 105.2)
- moved J6 0.42 mm to (75.0, 105.2)
- moved J7 0.42 mm to (75.0, 103.8)
- moved J8 0.42 mm to (58.0, 138.8)
- moved J9 0.42 mm to (58.0, 105.2)
Connections:
- net Net-(J3-In) renamed /SHORT
Routing:
- net /SHORT: track 6.25 -> 5.11 mm
- net Net-(J8-In): track 54.5 -> 53.7 mm
Other:
- board text added: "0"
- board text added: "0 mm"
- board text added: "0.01 mm"
- board text added: "0.0152 mm"
- board text added: "0.02"
- board text added: "0.035 mm"
- board text added: "0.2104 mm"
- board text added: "1"
- board text added: "1.065 mm"
- board text added: "1x 7628"
- board text added: "3.3"
- board text added: "4.4"
- board text added: "4.6"
- board text added: "B.Cu"
- board text added: "B.Mask"
- board text added: "B.Paste"
- board text added: "B.Silkscreen"
- board text added: "Bottom Silk Screen"
- board text added: "Bottom Solder Mask"
- board text added: "Bottom Solder Paste"
- board text added: "Color"
- board text added: "Core"
- board text added: "Dielectric"
- board text added: "Epsilon R"
- board text added: "F.Cu"
- board text added: "F.Mask"
- board text added: "F.Paste"
- board text added: "F.Silkscreen"
- board text added: "FR4 natural"
- board text added: "In1.Cu"
- board text added: "In2.Cu"
- board text added: "Layer Name"
- board text added: "Loss Tangent"
- board text added: "Material"
- board text added: "Not specified"
- board text added: "Thickness (mm)"
- board text added: "Top Silk Screen"
- board text added: "Top Solder Mask"
- board text added: "Top Solder Paste"
- board text added: "Type"
- board text added: "copper"
- board text added: "core"
- board text added: "prepreg"
