File: TRL_fixture_JLC04161H-7628.kicad_sch (KiCad schematic)
At the start: 11 parts, among them J1 142-0761-861, J2 142-0761-861, J3 142-0761-861, J4 142-0761-861, J5 142-0761-861, J6 142-0761-861, J7 142-0761-861, J8 142-0761-861, J9 142-0761-861

Commit message: TRL fixture DRC clean
Connections:
- net SHORT: now reaches J3.1 (In), NT1.2
Changed lines of the file:
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@@
 		)
 	)
-	(text_box "Calculated the following using Saturn PCB Toolkit:\n- Targeting JLC04161H-7628, 50ohm single-ended L1->L2 reference uStrip\n- Prepreg thickness 0.2104mm w/ relative permitivitty = 4.4\n- 50ohm trace width = 0.35mm.\n- Effective permitivitty for uStrip is 3.1408\n- Velocity Factor is 0.564\n- 90deg line at 6GHz is 7.048mm\n- 90deg line at 1GHz is 42.29mm"
+	(text_box "Calculated the following using Saturn PCB Toolkit:\n- Targeting JLC04161H-7628, 50ohm single-ended L1->L2 reference uStrip\n- Prepreg thickness 0.2104mm w/ relative permitivitty = 4.4\n- 50ohm trace width = 0.35mm.\n- Effective permitivitty for uStrip is 3.1408\n- Velocity Factor is 0.564\n- 90deg line at 6GHz is 7.048mm ~> 7mm\n- 90deg line at 1GHz is 42.29mm ~> 42mm"
 		(exclude_from_sim no)
 		(at 116.84 53.34 0)
@@
 		)
 	)
+	(label "SHORT"
+		(at 66.04 63.5 0)
+		(effects
+			(font
+				(size 1.27 1.27)
+			)
+			(justify left bottom)
+		)
+	)
+	(netclass_flag ""
+		(length 2.54)
+		(shape round)
+		(at 64.77 63.5 180)
+		(fields_autoplaced yes)
+		(effects
+			(font
+				(size 1.27 1.27)
+			)
+			(justify right bottom)
+		)
+		(property "Netclass" "clsSHORTED"
+			(at 65.4685 66.04 0)
+			(effects
+				(font
+					(size 1.27 1.27)
+				)
+				(justify left)
+			)
+		)
+		(property "Component Class" ""
+			(at 17.78 31.75 0)
+			(effects
+				(font
+					(size 1.27 1.27)
+					(italic yes)
+				)
+			)
+		)
+	)
